File: PCB_PROY_FINAL/RS485.kicad_sch (KiCad schematic)
At the start: 4 parts, among them IC4 SN75176BP

Commit message: Last update pcb
Parts:
- removed C4, C5: 1nF, PCM_JLCPCB:C_0402, symbol PCM_JLCPCB-Capacitors:0402,1nF
- removed D4: SM712, SOT95P240X115-3N, symbol SamacSys_Parts:SM712
- added D1: SM712_SOT23, Package_TO_SOT_SMD:SOT-23, symbol Diode:SM712_SOT23
- IC4: LCSC (none) -> C5215
Connections:
- net GND: now also D1.3 (common)
- net A renamed RS485_A
- net RS485_A: now also D1.1 (A1)
- net B renamed RS485_B
- net RS485_B: now also D1.2 (A2)
- net RTS renamed RS485_RTS
- net RX renamed RS485_RX_IN
- net TX renamed RS485_TX_OUT
- net V3.3 renamed +3.3V
