File: PCB_PROY_FINAL/KICADESPCONEX.kicad_sch (KiCad schematic)
At the start: 36 parts, among them IC1 USBLC6-2SC6, IC2 ESP32-S3-WROOM-1-N16, J1 Connector, USB-TYPE-C-16P

Commit message: Last update pcb
Parts:
- removed ADC/IO, DIGITAL_I/O: 1712805, SamacSys_Parts:1712805, symbol SamacSys_Parts:1712805
- removed C1, C10: 22uF, PCM_JLCPCB:C_0603, symbol PCM_JLCPCB-Capacitors:0603,22uF
- removed C15, C16: 1uF, PCM_JLCPCB:C_0402, symbol PCM_JLCPCB-Capacitors:0402,1uF
- removed C2, C3, C7, C9: 100nF, PCM_JLCPCB:C_0402, symbol PCM_JLCPCB-Capacitors:0402,100nF
- removed D10, D11, D12, D5, D6, D7, D8, D9: SMF3.3, SamacSys_Parts:SOD3718X108N, symbol SamacSys_Parts:SMF3.3
- removed IC1: USBLC6-2SC6, SamacSys_Parts:SOT95P280X145-6N, symbol SamacSys_Parts:USBLC6-2SC6
- removed LED1, LED2, LED3, LED4: KT-0603R, LEDC1608X70N, symbol SamacSys_Parts:KT-0603R
- removed R11, R3, R4, R5: 220Ω, PCM_JLCPCB:R_0402, symbol PCM_JLCPCB-Resistors:0402,220Ω
- removed R7: 4.7kΩ, PCM_JLCPCB:R_0402, symbol PCM_JLCPCB-Resistors:0402,4.7kΩ
- removed Reset1: XKB5858-W-TP, SamacSys_Parts:XKB5858WTP, symbol SamacSys_Parts:XKB5858-W-TP
- added C1: 22uF, PCM_JLCPCB:C_0805, symbol PCM_JLCPCB-Capacitors:0805,22uF
- added C10, C17, C7, C9: 100nF, PCM_JLCPCB:C_0603, symbol PCM_JLCPCB-Capacitors:0603,100nF
- added C16: 22uF, PCM_JLCPCB:C_1206, symbol PCM_JLCPCB-Capacitors:1206,22uF
- added R11: 4.7kΩ, PCM_JLCPCB:R_1206, symbol PCM_JLCPCB-Resistors:1206,4.7kΩ
- added SW1: SW_Push, SamacSys_Parts:XKB5858WTP, symbol Switch:SW_Push
- added U1: USBLC6-2SC6, Package_TO_SOT_SMD:SOT-23-6, symbol Power_Protection:USBLC6-2SC6
- IC2: LCSC (none) -> C2913199
- R1: LCSC C25744 -> C4139000
- R6, R8: LCSC C25105 -> C2122351
Connections:
- net D+: now also R8.1; no longer R6.1
- net D-: now also R6.2; no longer R8.1
- net EN: now also C10.1, SW1.2
- net GND: now also C1.2, C10.2, C16.2, C17.2, C7.2, C9.2, SW1.1, U1.2 (GND)
- net at J1.A7 (D-), J1.B7 (D-): now also U1.1 (I/O1)
- net at J1.A6 (D+), J1.B6 (D+): now also U1.3 (I/O2)
- net at R8.2: now also U1.4 (I/O2)
- net RTS renamed ESP_RTS
- net RX renamed ESP_RX_IN
- net TX renamed ESP_TX_OUT
- net USB-V renamed +5VD
- net +5VD: now also C1.1, C7.1, U1.5 (VBUS)
- net VDD33 renamed +3.3V
- net +3.3V: now also C16.1, C17.1, C9.1, R11.1; no longer IC2.27 (IO0)
- new net: R6.1, U1.6 (I/O1)
- new net: IC2.27 (IO0), R11.2
- no-connect marks 23 -> 20
Other:
- moved on the sheet: IC2, J1, R1, R10, R6, R8, R9

Commit message: new changes
Parts:
- removed C1: 22uF, PCM_JLCPCB:C_0805, symbol PCM_JLCPCB-Capacitors:0805,22uF
- removed C7: 100nF, PCM_JLCPCB:C_0603, symbol PCM_JLCPCB-Capacitors:0603,100nF
- removed J1: Connector, USB-TYPE-C-16P, PCM_JLCPCB:TYPE-C-SMD_HX-TYPE-C-16PIN, symbol PCM_JLCPCB-Extended:Connector, USB-TYPE-C-16P
- removed R10, R9: 5.1kΩ, PCM_JLCPCB:R_0805, symbol PCM_JLCPCB-Resistors:0805,5.1kΩ
- removed R6, R8: 33Ω, PCM_JLCPCB:R_0402, symbol PCM_JLCPCB-Resistors:0402,33Ω
- removed U1: USBLC6-2SC6, Package_TO_SOT_SMD:SOT-23-6, symbol Power_Protection:USBLC6-2SC6
- added D4, D5, D7, D8: SMF3.3, SamacSys_Parts:SOD3718X108N, symbol SamacSys_Parts:SMF3.3
- added R2, R3, R4, R5: 220Ω, PCM_JLCPCB:R_0603, symbol PCM_JLCPCB-Resistors:0603,220Ω
Connections:
- net DI/O15: now also D4.1 (K)
- net DI/O16: now also D5.1 (K)
- net DI/O17: now also D7.1 (K)
- net DI/O18: now also D8.1 (K)
- net GND: now also D4.2 (A), D5.2 (A), D7.2 (A), D8.2 (A)
- net LED1: now also R2.1
- net LED2: now also R3.1
- net LED3: now also R4.1
- net LED4: now also R5.1
- net D+ renamed ESP_D+
- net D- renamed ESP_D-
- new net LED_BIT0_ERROR_CASE: R5.2
- new net LED_BIT1_ERROR_CASE: R4.2
- new net LED_BIT2_ERROR_CASE: R3.2
- new net LED_ESPWORKING: R2.2
- no-connect marks 20 -> 18
Other:
- moved on the sheet: C10, C16, C17, C9, IC2, R1, R11, SW1

Commit message: Update
Parts:
- removed R2, R3, R4, R5: 220Ω, PCM_JLCPCB:R_0603, symbol PCM_JLCPCB-Resistors:0603,220Ω
- added Q4, Q5, Q6, Q7: MMBFJ211, SOT95P251X112-3N, symbol SamacSys_Parts:MMBFJ211
- added R12, R13, R14, R7: 10kΩ, PCM_JLCPCB:R_1206, symbol PCM_JLCPCB-Resistors:1206,10kΩ
- added R15, R16, R17, R18: 330Ω, PCM_JLCPCB:R_1206, symbol PCM_JLCPCB-Resistors:1206,330Ω
- added R2, R3, R4, R5: 1kΩ, PCM_JLCPCB:R_1206, symbol PCM_JLCPCB-Resistors:1206,1kΩ
Connections:
- net GND: now also Q4.2 (S), Q5.2 (S), Q6.2 (S), Q7.2 (S), R2.2, R3.2, R4.2, R5.2
- net LED1: now also R7.1
- net LED2: now also R12.1
- net LED3: now also R13.1
- net LED4: now also R14.2
- net LED_BIT0_ERROR_CASE: now also R18.1
- net LED_BIT1_ERROR_CASE: now also R17.1
- net LED_BIT2_ERROR_CASE: now also R16.1
- net LED_ESPWORKING: now also R15.1
- new net: Q5.1 (D), R17.2
- new net: Q5.3 (G), R13.2, R4.1
- new net: Q4.3 (G), R2.1, R7.2
- new net: Q6.3 (G), R12.2, R3.1
- new net: Q7.3 (G), R14.1, R5.1
- new net: Q4.1 (D), R15.2
- new net: Q7.1 (D), R18.2
- new net: Q6.1 (D), R16.2
Other:
- moved on the sheet: C10, C16, C17, C9, D4, D5, D7, D8, IC2, R1, R11, SW1
